Commit message: new urdf file and packages

File: asseyend/urdf/asseyend.urdf (robot description, URDF)
Before this commit: robot asseyend, 8 links, 7 joints
Links:
- added link baselink, mass 0.84715; collision mesh filename=package://asseyrot/meshes/base_link.STL; visual mesh filename=package://asseyrot/meshes/base_link.STL
- added link r1, mass 1.2687; collision mesh filename=package://asseyrot/meshes/r1.STL; visual mesh filename=package://asseyrot/meshes/r1.STL
Joints:
- added joint asdf: type fixed, parent base_link, child baselink, origin xyz=0 -0.7 0.0 rpy=0 0 0.32037, axis 0 0 1
- added joint mtr1: type continuous, parent baselink, child r1, origin xyz=-0.069094 0.10314 0.06 rpy=0 0 0.32037, axis 0 0 1

File: asseyrot/urdf/asseyrot.urdf (robot description, URDF)
Before this commit: robot asseyrot, 2 links, 1 joints
Links:
- removed link base_link
- added link baselink, mass 0.84715; collision mesh filename=package://asseyrot/meshes/base_link.STL; visual mesh filename=package://asseyrot/meshes/baselink.STL
Joints:
- added joint asdf: type fixed, parent base_link, child baselink, origin xyz=-0.069094 -1.10314 0.06 rpy=0 0 0.32037, axis 0 0 1
- joint mtr1: parent base_link -> baselink
